File: pcb/rev.A1/rgb2ypbpr.kicad_pcb (KiCad board)
At the start: 2 copper layers, 70.8 x 89.2 mm, 49 parts, among them J1 SCART-F, J10 USB_B_Micro, J3 Conn_01x05, J4 Conn_01x03, J5 RCJ-014, J6 RCJ-014, J7 RCJ-014, J8 RCJ-014, J9 RCJ-014, Q1 BC549B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

Commit message: pcb rev.A1: replace TO-92_Inline footprint with TO-92
Parts:
- Q1, Q2, Q3, Q4, Q5, Q6, Q7: footprint Package_TO_SOT_THT:TO-92_Inline -> Package_TO_SOT_THT:TO-92
Routing:
- net Net-(Q6-Pad1): track 12.3 -> 14.0 mm
- net Net-(Q4-Pad2): track 24.6 -> 23.2 mm
- net Net-(Q2-Pad2): track 9.06 -> 10.3 mm
- net Net-(Q1-Pad2): track 9.20 -> 10.5 mm
- net Net-(Q6-Pad2): track 10.4 -> 9.12 mm
- net Net-(Q4-Pad1): track 23.9 -> 24.7 mm
