File: pcb/rev.A1/rgb2ypbpr.sch (KiCad schematic (older format))
At the start: 49 parts, among them J1 SCART-F, J10 USB_B_Micro, J3 Conn_01x05, J4 Conn_01x03, J5 RCJ-014, J6 RCJ-014, J7 RCJ-014, J8 RCJ-014, J9 RCJ-014, Q1 BC549B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

Commit message: pcb rev.A1: replace TO-92_Inline footprint with TO-92
Parts:
- Q1, Q2, Q3, Q4, Q5, Q6, Q7: footprint Package_TO_SOT_THT:TO-92_Inline -> Package_TO_SOT_THT:TO-92
Changed lines of the file:
@@
 F 0 "Q6" H 4840 2463 39  0000 L CNN
 F 1 "BC549B" H 4840 2388 39  0000 L CNN
-F 2 "Package_TO_SOT_THT:TO-92_Inline" H 4850 2525 50  0001 C CNN
+F 2 "Package_TO_SOT_THT:TO-92" H 4850 2525 50  0001 C CNN
 F 3 "~" H 4650 2425 50  0001 C CNN
 	1    4650 2425
@@
 F 0 "Q7" H 5615 2263 39  0000 L CNN
 F 1 "BC549B" H 5615 2188 39  0000 L CNN
-F 2 "Package_TO_SOT_THT:TO-92_Inline" H 5625 2325 50  0001 C CNN
+F 2 "Package_TO_SOT_THT:TO-92" H 5625 2325 50  0001 C CNN
 F 3 "~" H 5425 2225 50  0001 C CNN
 	1    5425 2225
@@
 F 0 "Q5" H 7265 3438 39  0000 L CNN
 F 1 "BC549B" H 7265 3363 39  0000 L CNN
-F 2 "Package_TO_SOT_THT:TO-92_Inline" H 7275 3500 50  0001 C CNN
+F 2 "Package_TO_SOT_THT:TO-92" H 7275 3500 50  0001 C CNN
 F 3 "~" H 7075 3400 50  0001 C CNN
 	1    7075 3400
@@
 F 0 "Q4" H 6390 3463 39  0000 L CNN
 F 1 "BC549B" H 6390 3388 39  0000 L CNN
-F 2 "Package_TO_SOT_THT:TO-92_Inline" H 6400 3525 50  0001 C CNN
+F 2 "Package_TO_SOT_THT:TO-92" H 6400 3525 50  0001 C CNN
 F 3 "~" H 6200 3425 50  0001 C CNN
 	1    6200 3425
@@
 F 0 "Q1" H 5740 5388 39  0000 L CNN
 F 1 "BC549B" H 5740 5313 39  0000 L CNN
-F 2 "Package_TO_SOT_THT:TO-92_Inline" H 5750 5450 50  0001 C CNN
+F 2 "Package_TO_SOT_THT:TO-92" H 5750 5450 50  0001 C CNN
 F 3 "~" H 5550 5350 50  0001 C CNN
 	1    5550 5350
@@
 F 0 "Q2" H 5740 4413 39  0000 L CNN
 F 1 "BC549B" H 5740 4338 39  0000 L CNN
-F 2 "Package_TO_SOT_THT:TO-92_Inline" H 5750 4475 50  0001 C CNN
+F 2 "Package_TO_SOT_THT:TO-92" H 5750 4475 50  0001 C CNN
 F 3 "~" H 5550 4375 50  0001 C CNN
 	1    5550 4375
@@
 F 0 "Q3" H 4740 3913 39  0000 L CNN
 F 1 "BC549B" H 4740 3838 39  0000 L CNN
-F 2 "Package_TO_SOT_THT:TO-92_Inline" H 4750 3975 50  0001 C CNN
+F 2 "Package_TO_SOT_THT:TO-92" H 4750 3975 50  0001 C CNN
 F 3 "~" H 4550 3875 50  0001 C CNN
 	1    4550 3875
